File: KiCad_prj/mosfet_driver/mosfet_driver.kicad_sch (KiCad schematic)
At the start: 22 parts, among them J1 KLS S1G03C, J2 KLS S1G03C, J3 KLS S1G03C, J4 KLS S1G02C, J5 KLS S1G02C

Commit message: Mosfet driver v rev. 1.0 odeslan do vyroby
Parts:
- J1, J2, J3, J4, J5: now left out of the parts list
- R1, R2: JLCPCB Part # (none) -> C17477
- TP1, TP10, TP11, TP12, TP13, TP2, TP3, TP4, TP5, TP6, TP7, TP8, TP9: value TestPoint -> D1MM; now left out of the parts list
