File: KiCad_prj/mosfet_driver/supply.kicad_sch (KiCad schematic)
At the start: 4 parts, among them U1 MGJ2D051505SC, U2 MGJ2D051505SC

Commit message: Mosfet driver v rev. 1.0 odeslan do vyroby
Parts:
- C1, C2: JLCPCB Part # (none) -> C28233
- U1, U2: now left out of the parts list
Changed lines of the file:
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@@
 		(unit 1)
 		(exclude_from_sim no)
-		(in_bom yes)
+		(in_bom no)
 		(on_board yes)
 		(dnp no)
@@
 		)
 		(property "Description" "5.2kVDC Isolated 2W Gate Drive, 5V Vin, +15V/-5V Vout"
+			(at 139.7 106.68 0)
+			(effects
+				(font
+					(size 1.27 1.27)
+				)
+				(hide yes)
+			)
+		)
+		(property "JLCPCB Part #" ""
 			(at 139.7 106.68 0)
 			(effects
@@
 		(unit 1)
 		(exclude_from_sim no)
-		(in_bom yes)
+		(in_bom no)
 		(on_board yes)
 		(dnp no)
@@
 		)
 		(property "Description" "5.2kVDC Isolated 2W Gate Drive, 5V Vin, +15V/-5V Vout"
+			(at 139.7 60.96 0)
+			(effects
+				(font
+					(size 1.27 1.27)
+				)
+				(hide yes)
+			)
+		)
+		(property "JLCPCB Part #" ""
 			(at 139.7 60.96 0)
 			(effects
@@
 			)
 		)
+		(property "JLCPCB Part #" "C28233"
+			(at 115.57 59.69 0)
+			(effects
+				(font
+					(size 1.27 1.27)
+				)
+				(hide yes)
+			)
+		)
 		(pin "1"
 		)
@@
 			(at 115.57 105.41 0)
 			(effects
+				(font
+					(size 1.27 1.27)
+				)
+				(hide yes)
+			)
+		)
+		(property "JLCPCB Part #" "C28233"
+			(at 115.57 105.41 0)
+			(effects
