File: KiCad_prj/generator_strme_hrany_smd/generator_strme_hrany_smd.kicad_pcb (KiCad board)
At the start: 2 copper layers, 48 x 140 mm, 43 parts, among them J1 Barrel_Jack_Switch, J2 2EDGRC-5.08-03P, J3 Conn_Coaxial, J4 2EDGRC-5.08-03P, J5 Conn_Coaxial, SW1 SW_SPDT, SW2 SW_SPDT, SW3 SW_SPDT, U1 74HC14, U2 74HC14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

Commit message: Vyrobni data pro generator strme hrany
Routing:
- net /NEAR_END_N: track 40.3 -> 37.2 mm
- net /FAR_END_N: track 40.3 -> 37.4 mm
- net Net-(R10-Pad2): track 13.9 -> 16.1 mm
- net /FAR_END_P: track 58.2 -> 59.9 mm
- net /NEAR_END_P: track 58.1 -> 59.4 mm
