File: KiCad_prj/generator_strme_hrany_smd/generator_strme_hrany_smd.kicad_pcb (KiCad board)
At the start: 2 copper layers, 48 x 140 mm, 43 parts, among them J1 Barrel_Jack_Switch, J2 2EDGRC-5.08-03P, J3 Conn_Coaxial, J4 2EDGRC-5.08-03P, J5 Conn_Coaxial, SW1 SW_SPDT, SW2 SW_SPDT, SW3 SW_SPDT, U1 74HC14, U2 74HC14, U3 AMS1117-5.0

Commit message: pwm_generator 1.0 odeslan do vyroby
Parts:
- added R14: 22R, Resistor_SMD:R_0805_2012Metric, F.Cu at (126.4, 145.3)
- added R15: 22R, Resistor_SMD:R_0805_2012Metric, F.Cu at (128.9, 145.3)
- R1, R10, R11, R2, R3, R4, R5, R7, R8, R9: value 249R -> 220R
- U3: value AMS1117-5.0 -> AMS1117-3V3
Connections:
- RV2 pad 1: Net-(SW3-B) -> Net-(R14-Pad2)
- RV2 pad 4: Net-(SW3-B) -> Net-(R15-Pad2)
Routing:
- net Net-(SW3-B): track 13.2 -> 6.76 mm
- net Net-(R14-Pad2): track 0.00 -> 4.73 mm
- net Net-(R15-Pad2): track 0.00 -> 4.72 mm
