File: KiCad_prj/generator_strme_hrany_smd/generator_strme_hrany_smd.kicad_sch (KiCad schematic)
At the start: 43 parts, among them J1 Barrel_Jack_Switch, J2 2EDGRC-5.08-03P, J3 Conn_Coaxial, J4 2EDGRC-5.08-03P, J5 Conn_Coaxial, SW1 SW_SPDT, SW2 SW_SPDT, SW3 SW_SPDT, U1 74HC14, U2 74HC14, U3 AMS1117-5.0

Commit message: pwm_generator 1.0 odeslan do vyroby
Parts:
- added R14, R15: 22R, Resistor_SMD:R_0805_2012Metric, symbol Device:R
- R1, R10, R11, R2, R3, R4, R5, R7, R8, R9: value 249R -> 220R
- U3: value AMS1117-5.0 -> AMS1117-3V3
Connections:
- new net: R14.1, R15.1, SW3.2 (B)
- new net: R15.2, RV2.4
- new net: R14.2, RV2.1
Changed lines of the file:
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@@
 	(wire
 		(pts
-			(xy 237.49 30.48) (xy 237.49 38.1)
-		)
-		(stroke
-			(width 0)
-			(type default)
-		)
-	)
-	(wire
-		(pts
 			(xy 55.88 30.48) (xy 55.88 44.45)
 		)
@@
 	(wire
 		(pts
-			(xy 224.79 38.1) (xy 224.79 30.48)
-		)
-		(stroke
-			(width 0)
-			(type default)
-		)
-	)
-	(wire
-		(pts
 			(xy 45.72 30.48) (xy 55.88 30.48)
 		)
@@
 			)
 		)
-		(property "Value" "249R"
+		(property "Value" "220R"
 			(at 74.93 118.11 90)
 			(show_name no)
@@
 			)
 		)
-		(property "Value" "249R"
+		(property "Value" "220R"
 			(at 74.93 54.61 90)
 			(show_name no)
@@
 		(in_pos_files yes)
 		(dnp no)
-		(fields_autoplaced yes)
 		(property "Reference" "RV3"
-			(at 271.78 44.45 0)
+			(at 271.78 32.004 0)
 			(show_name no)
 			(do_not_autoplace no)
@@
 		)
 		(property "Value" "1k"
-			(at 271.78 46.99 0)
+			(at 271.78 34.036 0)
 			(show_name no)
 			(do_not_autoplace no)
@@
 			)
 		)
-		(property "Value" "249R"
+		(property "Value" "220R"
 			(at 74.93 40.64 90)
 			(show_name no)
@@
 			)
 		)
-		(property "Value" "249R"
+		(property "Value" "220R"
 			(at 74.93 104.14 90)
 			(show_name no)
@@
 			)
 		)
-		(property "Value" "249R"
+		(property "Value" "220R"
 			(at 74.93 68.58 90)
 			(show_name no)
@@
 			)
 		)
-		(property "Value" "249R"
+		(property "Value" "220R"
 			(at 74.93 132.08 90)
 			(show_name no)
@@
 	)
 	(symbol
+		(lib_id "Device:R")
+		(at 224.79 34.29 180)
+		(unit 1)
+		(body_style 1)
+		(exclude_from_sim no)
+		(in_bom yes)
+		(on_board yes)
+		(in_pos_files yes)
+		(dnp no)
+		(fields_autoplaced yes)
+		(property "Reference" "R15"
+			(at 227.33 33.0199 0)
+			(show_name no)
+			(do_not_autoplace no)
+			(effects
+				(font
+					(size 1.27 1.27)
+				)
+				(justify right)
+			)
+		)
+		(property "Value" "22R"
+			(at 227.33 35.5599 0)
+			(show_name no)
+			(do_not_autoplace no)
+			(effects
+				(font
+					(size 1.27 1.27)
+				)
+				(justify right)
+			)
+		)
+		(property "Footprint" "Resistor_SMD:R_0805_2012Metric"
+			(at 226.568 34.29 90)
+			(hide yes)
+			(show_name no)
+			(do_not_autoplace no)
+			(effects
+				(font
+					(size 1.27 1.27)
+				)
+			)
+		)
+		(property "Datasheet" ""
+			(at 224.79 34.29 0)
+			(hide yes)
+			(show_name no)
+			(do_not_autoplace no)
+			(effects
+				(font
+					(size 1.27 1.27)
+				)
+			)
+		)
+		(property "Description" "Resistor"
+			(at 224.79 34.29 0)
+			(hide yes)
+			(show_name no)
+			(do_not_autoplace no)
+			(effects
+				(font
+					(size 1.27 1.27)
+				)
+			)
+		)
+		(pin "1"
+		)
+		(pin "2"
+		)
+		(instances
+			(project "generator_strme_hrany_smd"
+				(path "/79be1a42-f11b-4399-83e4-46f5861d246a"
+					(reference "R15")
+					(unit 1)
+				)
+			)
+		)
+	)
+	(symbol
 		(lib_id "74xx:74HC14")
 		(at 63.5 163.83 0)
@@
 			)
 		)
-		(property "Value" "249R"
+		(property "Value" "220R"
 			(at 74.93 82.55 90)
 			(show_name no)
@@
 			)
 		)
-		(property "Value" "249R"
+		(property "Value" "220R"
 			(at 74.93 146.05 90)
 			(show_name no)
@@
 	)
 	(symbol
+		(lib_id "Device:R")
+		(at 237.49 34.29 180)
+		(unit 1)
+		(body_style 1)
+		(exclude_from_sim no)
+		(in_bom yes)
+		(on_board yes)
+		(in_pos_files yes)
+		(dnp no)
+		(fields_autoplaced yes)
+		(property "Reference" "R14"
+			(at 240.03 33.0199 0)
+			(show_name no)
+			(do_not_autoplace no)
+			(effects
+				(font
+					(size 1.27 1.27)
+				)
+				(justify right)
+			)
+		)
+		(property "Value" "22R"
+			(at 240.03 35.5599 0)
+			(show_name no)
+			(do_not_autoplace no)
+			(effects
+				(font
+					(size 1.27 1.27)
+				)
+				(justify right)
+			)
+		)
+		(property "Footprint" "Resistor_SMD:R_0805_2012Metric"
+			(at 239.268 34.29 90)
+			(hide yes)
+			(show_name no)
+			(do_not_autoplace no)
+			(effects
+				(font
+					(size 1.27 1.27)
+				)
+			)
+		)
+		(property "Datasheet" ""
+			(at 237.49 34.29 0)
+			(hide yes)
+			(show_name no)
+			(do_not_autoplace no)
+			(effects
+				(font
+					(size 1.27 1.27)
+				)
+			)
+		)
+		(property "Description" "Resistor"
+			(at 237.49 34.29 0)
+			(hide yes)
+			(show_name no)
+			(do_not_autoplace no)
+			(effects
+				(font
+					(size 1.27 1.27)
+				)
+			)
+		)
+		(pin "1"
+		)
+		(pin "2"
+		)
+		(instances
+			(project "generator_strme_hrany_smd"
+				(path "/79be1a42-f11b-4399-83e4-46f5861d246a"
+					(reference "R14")
+					(unit 1)
+				)
+			)
+		)
+	)
+	(symbol
 		(lib_id "power:GND")
 		(at 139.7 36.83 0)
@@
 		(in_pos_files yes)
 		(dnp no)
-		(fields_autoplaced yes)
 		(property "Reference" "RV2"
-			(at 227.33 34.29 0)
+			(at 227.33 20.066 0)
 			(show_name no)
 			(do_not_autoplace no)
@@
 		)
 		(property "Value" "1k"
-			(at 227.33 36.83 0)
+			(at 227.33 21.844 0)
 			(show_name no)
 			(do_not_autoplace no)
@@
 			)
 		)
-		(property "Value" "249R"
+		(property "Value" "220R"
 			(at 74.93 26.67 90)
 			(show_name no)
@@
 			)
 		)
-		(property "Value" "249R"
+		(property "Value" "220R"
 			(at 74.93 160.02 90)
 			(show_name no)
@@
 			)
 		)
-		(property "Value" "AMS1117-5.0"
+		(property "Value" "AMS1117-3V3"
 			(at 170.18 81.28 0)
 			(show_name no)
