File: KiCad_prj/power_bank/power_bank.kicad_pcb (KiCad board)
At the start: 2 copper layers, 130 x 60 mm, 80 parts, among them J1 svorkovnice, J2 svorkovnice, J3 vypinac, J4 vypinac, Q1 BC847BS, Q2 BC857BS, Q3 IRFR5305, Q4 IRFR4105, U1 LMR51625, U2 TPS564242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

Commit message: Oprava objednavaciho kodu u power_bank
Parts:
- moved R10 4.43 mm to (157.0, 106.7), turned to 180 degrees
Routing:
- net Net-(D3-A): track 32.1 -> 40.0 mm
- net /Battery/CHA_POS: track 168.3 -> 166.6 mm
Changed lines of the file:
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@@
 	(property "DESCR" "U_{in}: 20V až 50V; U_{out}: 5V; P: 10W")
 	(property "FILENAME" "pwbank")
-	(property "REVISION" "1.0")
+	(property "REVISION" "1.1")
 	(property "TITLE" "Power bank pro solární panel")
 	(net 0 "")
@@
 	(footprint "Resistor_SMD:R_0805_2012Metric"
 		(layer "F.Cu")
-		(at 160.843 108.839 90)
+		(at 156.972 106.68 180)
 		(descr "Resistor SMD 0805 (2012 Metric), square (rectangular) end terminal, IPC-7351 nominal, (Body size source: IPC-SM-782 page 72, https://www.pcb-3d.com/wordpress/wp-content/uploads/ipc-sm-782a_amendment_1_and_2.pdf), generated with kicad-footprint-generator")
 		(tags "resistor")
 		(property "Reference" "R10"
-			(at 0 -1.65 90)
+			(at -3.048 -3.048 0)
 			(layer "F.SilkS")
 			(effects
@@
 		)
 		(property "Value" "3k3"
-			(at 0 1.65 90)
+			(at 0 1.65 0)
 			(layer "F.Fab")
 			(effects
@@
 		)
 		(property "Datasheet" "~"
-			(at 0 0 90)
+			(at 0 0 0)
 			(layer "F.Fab")
 			(hide yes)
@@
 		)
 		(property "Description" "Resistor"
-			(at 0 0 90)
+			(at 0 0 0)
 			(layer "F.Fab")
 			(hide yes)
@@
 		(attr smd)
 		(fp_line
-			(start -0.227064 -0.735)
-			(end 0.227064 -0.735)
+			(start -0.227064 0.735)
+			(end 0.227064 0.735)
 			(stroke
 				(width 0.12)
@@
 		)
 		(fp_line
-			(start -0.227064 0.735)
-			(end 0.227064 0.735)
+			(start -0.227064 -0.735)
+			(end 0.227064 -0.735)
 			(stroke
 				(width 0.12)
@@
 		)
 		(fp_line
-			(start 1.68 -0.95)
-			(end 1.68 0.95)
+			(start 1.68 0.95)
+			(end -1.68 0.95)
 			(stroke
 				(width 0.05)
@@
 		)
 		(fp_line
-			(start -1.68 -0.95)
-			(end 1.68 -0.95)
+			(start 1.68 -0.95)
+			(end 1.68 0.95)
 			(stroke
 				(width 0.05)
@@
 		)
 		(fp_line
-			(start 1.68 0.95)
-			(end -1.68 0.95)
+			(start -1.68 0.95)
+			(end -1.68 -0.95)
 			(stroke
 				(width 0.05)
@@
 		)
 		(fp_line
-			(start -1.68 0.95)
-			(end -1.68 -0.95)
+			(start -1.68 -0.95)
+			(end 1.68 -0.95)
 			(stroke
 				(width 0.05)
@@
 		)
 		(fp_line
-			(start 1 -0.625)
-			(end 1 0.625)
+			(start 1 0.625)
+			(end -1 0.625)
 			(stroke
 				(width 0.1)
@@
 		)
 		(fp_line
-			(start -1 -0.625)
-			(end 1 -0.625)
+			(start 1 -0.625)
+			(end 1 0.625)
 			(stroke
 				(width 0.1)
@@
 		)
 		(fp_line
-			(start 1 0.625)
-			(end -1 0.625)
+			(start -1 0.625)
+			(end -1 -0.625)
 			(stroke
 				(width 0.1)
@@
 		)
 		(fp_line
-			(start -1 0.625)
-			(end -1 -0.625)
+			(start -1 -0.625)
+			(end 1 -0.625)
 			(stroke
 				(width 0.1)
@@
 		)
 		(fp_text user "${REFERENCE}"
-			(at 0 0 90)
+			(at 0 0 0)
 			(layer "F.Fab")
 			(effects
@@
 		)
 		(pad "1" smd roundrect
-			(at -0.9125 0 90)
+			(at -0.9125 0 180)
 			(size 1.025 1.4)
 			(layers "F.Cu" "F.Mask" "F.Paste")
@@
 		)
 		(pad "2" smd roundrect
-			(at 0.9125 0 90)
+			(at 0.9125 0 180)
 			(size 1.025 1.4)
 			(layers "F.Cu" "F.Mask" "F.Paste")
@@
 		(tags "capacitor")
 		(property "Reference" "C12"
-			(at 0 -1.68 90)
+			(at 0 -2.479 90)
 			(layer "F.SilkS")
 			(effects
@@
 		(tags "capacitor")
 		(property "Reference" "C10"
-			(at 0 -1.68 0)
+			(at 3.053 -2.794 0)
 			(layer "F.SilkS")
 			(effects
@@
 	)
 	(gr_text "+V_{BT2}<>VIN-GND"
-		(at 165.1 105.156 0)
+		(at 165.1 104.14 0)
 		(layer "F.SilkS")
 		(effects
@@
 	(segment
 		(start 179.766 93.345)
-		(end 179.766 88.519)
+		(end 175.575 97.536)
 		(width 0.762)
 		(layer "F.Cu")
@@
 	)
 	(segment
-		(start 156.017 106.299)
-		(end 156.017 107.95)
+		(start 156.017 111.826)
+		(end 156.017 109.474)
+		(width 0.762)
+		(layer "F.Cu")
+		(net 3)
+	)
+	(segment
+		(start 147.254 97.536)
+		(end 156.0595 106.3415)
 		(width 0.762)
 		(layer "F.Cu")
@@
 	)
 	(segment
-		(start 195.566 89.784)
-		(end 192.466 92.884)
+		(start 179.766 88.519)
+		(end 179.766 93.345)
 		(width 0.762)
 		(layer "F.Cu")
@@
 	)
 	(segment
-		(start 171.1935 97.536)
-		(end 175.575 97.536)
+		(start 156.017 109.474)
+		(end 156.017 106.7225)
+		(width 0.762)
+		(layer "F.Cu")
+		(net 3)
+	)
+	(segment
+		(start 195.566 89.784)
+		(end 192.466 92.884)
 		(width 0.762)
 		(layer "F.Cu")
@@
 	)
 	(segment
-		(start 156.017 109.474)
-		(end 156.017 107.95)
+		(start 175.575 97.536)
+		(end 164.592 97.536)
 		(width 0.762)
 		(layer "F.Cu")
@@
 	)
 	(segment
-		(start 182.466 90.384)
-		(end 189.966 90.384)
+		(start 156.0595 106.0685)
+		(end 156.0595 106.68)
 		(width 0.762)
 		(layer "F.Cu")
@@
 	)
 	(segment
-		(start 160.7795 107.95)
-		(end 171.1935 97.536)
+		(start 182.466 90.384)
+		(end 189.966 90.384)
 		(width 0.762)
 		(layer "F.Cu")
@@
 	)
 	(segment
-		(start 156.017 107.95)
-		(end 160.7795 107.95)
+		(start 156.017 106.7225)
+		(end 156.0595 106.68)
+		(width 0.762)
+		(layer "F.Cu")
+		(net 3)
+	)
+	(segment
+		(start 164.592 97.536)
+		(end 156.0595 106.0685)
 		(width 0.762)
 		(layer "F.Cu")
@@
 	)
 	(segment
-		(start 156.017 111.826)
-		(end 153.182 111.826)
+		(start 181.041 87.244)
+		(end 179.766 88.519)
 		(width 0.762)
 		(layer "F.Cu")
@@
 	)
 	(segment
-		(start 179.766 88.519)
-		(end 181.041 87.244)
+		(start 156.017 111.826)
+		(end 153.182 111.826)
 		(width 0.762)
 		(layer "F.Cu")
@@
 	)
 	(segment
-		(start 181.041 87.244)
-		(end 182.56 87.244)
+		(start 113.726 93.218)
+		(end 116.78 90.164)
 		(width 0.762)
 		(layer "F.Cu")
@@
 	)
 	(segment
-		(start 113.726 93.218)
-		(end 116.78 90.164)
+		(start 198.628 104.46)
+		(end 198.562 104.394)
 		(width 0.762)
 		(layer "F.Cu")
@@
 	)
 	(segment
-		(start 198.628 104.46)
-		(end 198.562 104.394)
+		(start 156.0595 106.3415)
+		(end 156.0595 106.68)
 		(width 0.762)
 		(layer "F.Cu")
@@
 	)
 	(segment
-		(start 156.017 111.826)
-		(end 156.017 107.95)
+		(start 113.726 94.5915)
+		(end 113.726 93.218)
 		(width 0.762)
 		(layer "F.Cu")
@@
 	)
 	(segment
-		(start 113.726 94.5915)
-		(end 113.726 93.218)
+		(start 182.56 87.244)
+		(end 181.041 87.244)
 		(width 0.762)
 		(layer "F.Cu")
@@
 	)
 	(segment
-		(start 147.254 97.536)
-		(end 156.017 106.299)
-		(width 0.762)
-		(layer "F.Cu")
-		(net 3)
-	)
-	(segment
 		(start 125.115 94.737)
 		(end 125.664 94.188)
@@
 	)
 	(segment
-		(start 175.575 97.536)
-		(end 179.766 93.345)
-		(width 0.762)
-		(layer "F.Cu")
-		(net 3)
-	)
-	(segment
 		(start 126.724 83.074)
 		(end 126.9835 83.074)
@@
 	)
 	(segment
-		(start 163.8675 112.776)
+		(start 160.16575 112.41375)
+		(end 162.56 114.808)
+		(width 0.762)
+		(layer "F.Cu")
+		(net 30)
+	)
+	(segment
+		(start 178.816 114.808)
+		(end 180.848 112.776)
+		(width 0.762)
+		(layer "F.Cu")
+		(net 30)
+	)
+	(segment
+		(start 160.16575 109.07425)
+		(end 160.16575 112.41375)
+		(width 0.762)
+		(layer "F.Cu")
+		(net 30)
+	)
+	(segment
+		(start 157.8845 106.793)
+		(end 160.16575 109.07425)
+		(width 0.762)
+		(layer "F.Cu")
+		(net 30)
+	)
+	(segment
+		(start 162.56 114.808)
+		(end 178.816 114.808)
+		(width 0.762)
+		(layer "F.Cu")
+		(net 30)
+	)
+	(segment
+		(start 180.848 112.776)
 		(end 186.116 112.776)
 		(width 0.762)
@@
 	)
 	(segment
-		(start 160.843 109.7515)
-		(end 163.8675 112.776)
+		(start 157.8845 106.68)
+		(end 157.8845 106.793)
 		(width 0.762)
 		(layer "F.Cu")
