File: KiCad_prj/pwm_generator/shaper.kicad_sch (KiCad schematic)
At the start: 32 parts, among them U6 OPA197xDBV, U7 OPA197xDBV, U8 OPA197xDBV, U9 OPA197xDBV

Commit message: Pocatek prace na DPS
Parts:
- renumbered C10 to C11, C11 to C12, C12 to C13, C13 to C14, C14 to C15, C15 to C16, C16 to C17, C17 to C18, C18 to C19
Connections:
- net SIGNAL_REF_INV renamed ~{SIGNAL_REF}

Commit message: precislovani
Parts:
- renumbered C18 to C17, C19 to C18, C17 to C19, C11 to C20, C13 to C21, C12 to C22, C14 to C23, D3 to D1, D4 to D2, D5 to D3, D6 to D4, D1 to D5, D2 to D6, R22 to R16, R24 to R17, R23 to R18, R20 to R19, R21 to R20, R25 to R21, R13 to R22, R14 to R23, R15 to R24, R19 to R25, R16 to R26, R17 to R27, R18 to R28, U8 to U6, U9 to U7, U6 to U8, U7 to U9

Commit message: Pridany testpointy a jlcpcb bom reference
Parts:
- added C34: 100n, Capacitor_SMD:C_0805_2012Metric, symbol Device:C
- added R42: 1k, Resistor_SMD:R_0805_2012Metric, symbol Device:R
- C15, C16, C17, C18, C20, C21, C22, C23: JLCPCB Part # (none) -> C49678
- C19: JLCPCB Part # (none) -> C1790
- D1, D2, D3, D4: value LL4148 -> 1N4148WS; footprint Diode_SMD:D_MiniMELF -> Diode_SMD:D_SOD-323; JLCPCB Part # (none) -> C2128
- D5, D6: JLCPCB Part # (none) -> C41410795
- R16, R17, R19, R20, R23, R24, R26, R27, R28: JLCPCB Part # (none) -> C17414
- R18, R21: JLCPCB Part # (none) -> C17513
- R22: value 2k5 -> 1k5; JLCPCB Part # (none) -> C4310
- R25: JLCPCB Part # (none) -> C17633
- U6, U7, U8, U9: JLCPCB Part # (none) -> C221351
Connections:
- net ACDC: now also R42.1; no longer R22.1
- net GND: now also C34.1
- net at R22.2, R23.1: now also C34.2
- new net: R22.1, R42.2
Other:
- moved on the sheet: R22

Commit message: Doplnene testovaci body a popisky
Parts:
- renumbered C34 to C20, C20 to C21, C21 to C22, C22 to C23, C23 to C24, D1 to D2, D2 to D3, D3 to D4, D4 to D5, D5 to D6, D6 to D7, R16 to R17, R17 to R18, R18 to R19, R19 to R20, R42 to R21, R20 to R22, R21 to R23, R22 to R24, R23 to R25, R24 to R26, R25 to R27, R26 to R28, R27 to R29, R28 to R30
