File: KiCad_prj/pwm_generator/twg.kicad_sch (KiCad schematic)
At the start: 12 parts, among them U4 OPA365xxDBV, U5 TLV3501AIDBV

Commit message: Priprava na prezentaci Kicad
Parts:
- C7: value 33n -> 3n3
Changed lines of the file:
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@@
 			)
 		)
-		(property "Value" "33n"
+		(property "Value" "3n3"
 			(at 162.56 91.44 90)
 			(show_name no)

Commit message: Pocatek prace na DPS
Parts:
- renumbered C9 to C10, C5 to C6, C6 to C7, C7 to C8, C8 to C9
Connections:
- net SAMPLING renamed ~{SAMPLING}
Changed lines of the file:
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@@
 		)
 	)
-	(hierarchical_label "SAMPLING"
+	(hierarchical_label "~{SAMPLING}"
 		(shape output)
 		(at 102.87 128.27 180)
@@
 		(dnp no)
 		(fields_autoplaced yes)
-		(property "Reference" "#PWR020"
+		(property "Reference" "#PWR021"
 			(at 146.05 54.61 0)
 			(hide yes)
@@
 			(project "pwm_generator"
 				(path "/8c5142ba-d623-44cf-91e0-639551b20541/749c89d5-b92c-45c1-9dff-9c60a81aaaf0"
-					(reference "#PWR020")
+					(reference "#PWR021")
 					(unit 1)
 				)
@@
 		(dnp no)
 		(fields_autoplaced yes)
-		(property "Reference" "#PWR021"
+		(property "Reference" "#PWR022"
 			(at 129.54 52.07 0)
 			(hide yes)
@@
 			(project "pwm_generator"
 				(path "/8c5142ba-d623-44cf-91e0-639551b20541/749c89d5-b92c-45c1-9dff-9c60a81aaaf0"
-					(reference "#PWR021")
+					(reference "#PWR022")
 					(unit 1)
 				)
@@
 		(dnp no)
 		(fields_autoplaced yes)
-		(property "Reference" "#PWR025"
+		(property "Reference" "#PWR026"
 			(at 115.57 119.38 0)
 			(hide yes)
@@
 			(project "pwm_generator"
 				(path "/8c5142ba-d623-44cf-91e0-639551b20541/749c89d5-b92c-45c1-9dff-9c60a81aaaf0"
-					(reference "#PWR025")
+					(reference "#PWR026")
 					(unit 1)
 				)
@@
 		(dnp no)
 		(fields_autoplaced yes)
-		(property "Reference" "C8"
+		(property "Reference" "C9"
 			(at 125.73 111.76 90)
 			(show_name no)
@@
 			(project "pwm_generator"
 				(path "/8c5142ba-d623-44cf-91e0-639551b20541/749c89d5-b92c-45c1-9dff-9c60a81aaaf0"
-					(reference "C8")
+					(reference "C9")
 					(unit 1)
 				)
@@
 		(dnp no)
 		(fields_autoplaced yes)
-		(property "Reference" "#PWR026"
+		(property "Reference" "#PWR027"
 			(at 129.54 144.78 0)
 			(hide yes)
@@
 			(project "pwm_generator"
 				(path "/8c5142ba-d623-44cf-91e0-639551b20541/749c89d5-b92c-45c1-9dff-9c60a81aaaf0"
-					(reference "#PWR026")
+					(reference "#PWR027")
 					(unit 1)
 				)
@@
 		(dnp no)
 		(fields_autoplaced yes)
-		(property "Reference" "#PWR027"
+		(property "Reference" "#PWR028"
 			(at 132.08 144.78 0)
 			(hide yes)
@@
 			(project "pwm_generator"
 				(path "/8c5142ba-d623-44cf-91e0-639551b20541/749c89d5-b92c-45c1-9dff-9c60a81aaaf0"
-					(reference "#PWR027")
+					(reference "#PWR028")
 					(unit 1)
 				)
@@
 		(dnp no)
 		(fields_autoplaced yes)
-		(property "Reference" "#PWR022"
+		(property "Reference" "#PWR023"
 			(at 119.38 72.39 0)
 			(hide yes)
@@
 			(project "pwm_generator"
 				(path "/8c5142ba-d623-44cf-91e0-639551b20541/749c89d5-b92c-45c1-9dff-9c60a81aaaf0"
-					(reference "#PWR022")
+					(reference "#PWR023")
 					(unit 1)
 				)
@@
 		(dnp no)
 		(fields_autoplaced yes)
-		(property "Reference" "#PWR024"
+		(property "Reference" "#PWR025"
 			(at 132.08 121.92 0)
 			(hide yes)
@@
 			(project "pwm_generator"
 				(path "/8c5142ba-d623-44cf-91e0-639551b20541/749c89d5-b92c-45c1-9dff-9c60a81aaaf0"
-					(reference "#PWR024")
+					(reference "#PWR025")
 					(unit 1)
 				)
@@
 		(dnp no)
 		(fields_autoplaced yes)
-		(property "Reference" "C9"
+		(property "Reference" "C10"
 			(at 166.37 133.3499 0)
 			(show_name no)
@@
 			(project "pwm_generator"
 				(path "/8c5142ba-d623-44cf-91e0-639551b20541/749c89d5-b92c-45c1-9dff-9c60a81aaaf0"
-					(reference "C9")
+					(reference "C10")
 					(unit 1)
 				)
@@
 		(dnp no)
 		(fields_autoplaced yes)
-		(property "Reference" "#PWR028"
+		(property "Reference" "#PWR029"
 			(at 162.56 144.78 0)
 			(hide yes)
@@
 			(project "pwm_generator"
 				(path "/8c5142ba-d623-44cf-91e0-639551b20541/749c89d5-b92c-45c1-9dff-9c60a81aaaf0"
-					(reference "#PWR028")
+					(reference "#PWR029")
 					(unit 1)
 				)
@@
 		(dnp no)
 		(fields_autoplaced yes)
-		(property "Reference" "C5"
+		(property "Reference" "C6"
 			(at 139.7 44.45 90)
 			(show_name no)
@@
 			(project "pwm_generator"
 				(path "/8c5142ba-d623-44cf-91e0-639551b20541/749c89d5-b92c-45c1-9dff-9c60a81aaaf0"
-					(reference "C5")
+					(reference "C6")
 					(unit 1)
 				)
@@
 		(dnp no)
 		(fields_autoplaced yes)
-		(property "Reference" "C6"
+		(property "Reference" "C7"
 			(at 115.57 60.9599 0)
 			(show_name no)
@@
 			(project "pwm_generator"
 				(path "/8c5142ba-d623-44cf-91e0-639551b20541/749c89d5-b92c-45c1-9dff-9c60a81aaaf0"
-					(reference "C6")
+					(reference "C7")
 					(unit 1)
 				)
@@
 		(dnp no)
 		(fields_autoplaced yes)
-		(property "Reference" "C7"
+		(property "Reference" "C8"
 			(at 162.56 88.9 90)
 			(show_name no)
@@
 			(project "pwm_generator"
 				(path "/8c5142ba-d623-44cf-91e0-639551b20541/749c89d5-b92c-45c1-9dff-9c60a81aaaf0"
-					(reference "C7")
+					(reference "C8")
 					(unit 1)
 				)
@@
 		(in_pos_files yes)
 		(dnp no)
-		(property "Reference" "#PWR023"
+		(property "Reference" "#PWR024"
 			(at 146.05 74.93 0)
 			(hide yes)
@@
 			(project "pwm_generator"
 				(path "/8c5142ba-d623-44cf-91e0-639551b20541/749c89d5-b92c-45c1-9dff-9c60a81aaaf0"
-					(reference "#PWR023")
-					(unit 1)
-				)
+					(reference "#PWR024")
+					(unit 1)
+				)

Commit message: precislovani
Parts:
- renumbered C7 to C10, C9 to C11, C6 to C12, C8 to C13, C10 to C14, R8 to R11, R9 to R12, R10 to R13, R11 to R14, R12 to R15, U5 to U4, U4 to U5
Changed lines of the file:
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@@
 		(dnp no)
 		(fields_autoplaced yes)
-		(property "Reference" "#PWR021"
+		(property "Reference" "#PWR028"
 			(at 146.05 54.61 0)
 			(hide yes)
@@
 			(project "pwm_generator"
 				(path "/8c5142ba-d623-44cf-91e0-639551b20541/749c89d5-b92c-45c1-9dff-9c60a81aaaf0"
-					(reference "#PWR021")
+					(reference "#PWR028")
 					(unit 1)
 				)
@@
 		(dnp no)
 		(fields_autoplaced yes)
-		(property "Reference" "#PWR022"
+		(property "Reference" "#PWR027"
 			(at 129.54 52.07 0)
 			(hide yes)
@@
 			(project "pwm_generator"
 				(path "/8c5142ba-d623-44cf-91e0-639551b20541/749c89d5-b92c-45c1-9dff-9c60a81aaaf0"
-					(reference "#PWR022")
+					(reference "#PWR027")
 					(unit 1)
 				)
@@
 		(dnp no)
 		(fields_autoplaced yes)
-		(property "Reference" "#PWR026"
+		(property "Reference" "#PWR023"
 			(at 115.57 119.38 0)
 			(hide yes)
@@
 			(project "pwm_generator"
 				(path "/8c5142ba-d623-44cf-91e0-639551b20541/749c89d5-b92c-45c1-9dff-9c60a81aaaf0"
-					(reference "#PWR026")
+					(reference "#PWR023")
 					(unit 1)
 				)
@@
 		(dnp no)
 		(fields_autoplaced yes)
-		(property "Reference" "C9"
+		(property "Reference" "C11"
 			(at 125.73 111.76 90)
 			(show_name no)
@@
 			(project "pwm_generator"
 				(path "/8c5142ba-d623-44cf-91e0-639551b20541/749c89d5-b92c-45c1-9dff-9c60a81aaaf0"
-					(reference "C9")
+					(reference "C11")
 					(unit 1)
 				)
@@
 		(dnp no)
 		(fields_autoplaced yes)
-		(property "Reference" "R10"
+		(property "Reference" "R13"
 			(at 132.08 101.6 90)
 			(show_name no)
@@
 			(project "pwm_generator"
 				(path "/8c5142ba-d623-44cf-91e0-639551b20541/749c89d5-b92c-45c1-9dff-9c60a81aaaf0"
-					(reference "R10")
+					(reference "R13")
 					(unit 1)
 				)
@@
 		(dnp no)
 		(fields_autoplaced yes)
-		(property "Reference" "R11"
+		(property "Reference" "R14"
 			(at 162.56 101.6 90)
 			(show_name no)
@@
 			(project "pwm_generator"
 				(path "/8c5142ba-d623-44cf-91e0-639551b20541/749c89d5-b92c-45c1-9dff-9c60a81aaaf0"
-					(reference "R11")
+					(reference "R14")
 					(unit 1)
 				)
@@
 		(dnp no)
 		(fields_autoplaced yes)
-		(property "Reference" "U4"
+		(property "Reference" "U5"
 			(at 161.29 54.5398 0)
 			(show_name no)
@@
 			(project "pwm_generator"
 				(path "/8c5142ba-d623-44cf-91e0-639551b20541/749c89d5-b92c-45c1-9dff-9c60a81aaaf0"
-					(reference "U4")
+					(reference "U5")
 					(unit 1)
 				)
@@
 		(dnp no)
 		(fields_autoplaced yes)
-		(property "Reference" "R8"
+		(property "Reference" "R11"
 			(at 132.08 73.66 90)
 			(show_name no)
@@
 			(project "pwm_generator"
 				(path "/8c5142ba-d623-44cf-91e0-639551b20541/749c89d5-b92c-45c1-9dff-9c60a81aaaf0"
-					(reference "R8")
+					(reference "R11")
 					(unit 1)
 				)
@@
 		(dnp no)
 		(fields_autoplaced yes)
-		(property "Reference" "#PWR027"
+		(property "Reference" "#PWR024"
 			(at 129.54 144.78 0)
 			(hide yes)
@@
 			(project "pwm_generator"
 				(path "/8c5142ba-d623-44cf-91e0-639551b20541/749c89d5-b92c-45c1-9dff-9c60a81aaaf0"
-					(reference "#PWR027")
+					(reference "#PWR024")
 					(unit 1)
 				)
@@
 		(dnp no)
 		(fields_autoplaced yes)
-		(property "Reference" "R9"
+		(property "Reference" "R12"
 			(at 132.08 90.17 90)
 			(show_name no)
@@
 			(project "pwm_generator"
 				(path "/8c5142ba-d623-44cf-91e0-639551b20541/749c89d5-b92c-45c1-9dff-9c60a81aaaf0"
-					(reference "R9")
+					(reference "R12")
 					(unit 1)
 				)
@@
 		(dnp no)
 		(fields_autoplaced yes)
-		(property "Reference" "#PWR028"
+		(property "Reference" "#PWR026"
 			(at 132.08 144.78 0)
 			(hide yes)
@@
 			(project "pwm_generator"
 				(path "/8c5142ba-d623-44cf-91e0-639551b20541/749c89d5-b92c-45c1-9dff-9c60a81aaaf0"
-					(reference "#PWR028")
+					(reference "#PWR026")
 					(unit 1)
 				)
@@
 		(dnp no)
 		(fields_autoplaced yes)
-		(property "Reference" "#PWR023"
+		(property "Reference" "#PWR022"
 			(at 119.38 72.39 0)
 			(hide yes)
@@
 			(project "pwm_generator"
 				(path "/8c5142ba-d623-44cf-91e0-639551b20541/749c89d5-b92c-45c1-9dff-9c60a81aaaf0"
-					(reference "#PWR023")
+					(reference "#PWR022")
 					(unit 1)
 				)
@@
 		(dnp no)
 		(fields_autoplaced yes)
-		(property "Reference" "R12"
+		(property "Reference" "R15"
 			(at 162.56 119.38 90)
 			(show_name no)
@@
 			(project "pwm_generator"
 				(path "/8c5142ba-d623-44cf-91e0-639551b20541/749c89d5-b92c-45c1-9dff-9c60a81aaaf0"
-					(reference "R12")
+					(reference "R15")
 					(unit 1)
 				)
@@
 		(dnp no)
 		(fields_autoplaced yes)
-		(property "Reference" "C10"
+		(property "Reference" "C14"
 			(at 166.37 133.3499 0)
 			(show_name no)
@@
 			(project "pwm_generator"
 				(path "/8c5142ba-d623-44cf-91e0-639551b20541/749c89d5-b92c-45c1-9dff-9c60a81aaaf0"
-					(reference "C10")
+					(reference "C14")
 					(unit 1)
 				)
@@
 		(dnp no)
 		(fields_autoplaced yes)
-		(property "Reference" "U5"
+		(property "Reference" "U4"
 			(at 135.1981 118.11 0)
 			(show_name no)
@@
 			(project "pwm_generator"
 				(path "/8c5142ba-d623-44cf-91e0-639551b20541/749c89d5-b92c-45c1-9dff-9c60a81aaaf0"
-					(reference "U5")
+					(reference "U4")
 					(unit 1)
 				)
@@
 		(dnp no)
 		(fields_autoplaced yes)
-		(property "Reference" "#PWR029"
+		(property "Reference" "#PWR030"
 			(at 162.56 144.78 0)
 			(hide yes)
@@
 			(project "pwm_generator"
 				(path "/8c5142ba-d623-44cf-91e0-639551b20541/749c89d5-b92c-45c1-9dff-9c60a81aaaf0"
-					(reference "#PWR029")
+					(reference "#PWR030")
 					(unit 1)
 				)
@@
 		(dnp no)
 		(fields_autoplaced yes)
-		(property "Reference" "C6"
+		(property "Reference" "C12"
 			(at 139.7 44.45 90)
 			(show_name no)
@@
 			(project "pwm_generator"
 				(path "/8c5142ba-d623-44cf-91e0-639551b20541/749c89d5-b92c-45c1-9dff-9c60a81aaaf0"
-					(reference "C6")
+					(reference "C12")
 					(unit 1)
 				)
@@
 		(dnp no)
 		(fields_autoplaced yes)
-		(property "Reference" "C7"
+		(property "Reference" "C10"
 			(at 115.57 60.9599 0)
 			(show_name no)
@@
 			(project "pwm_generator"
 				(path "/8c5142ba-d623-44cf-91e0-639551b20541/749c89d5-b92c-45c1-9dff-9c60a81aaaf0"
-					(reference "C7")
+					(reference "C10")
 					(unit 1)
 				)
@@
 		(dnp no)
 		(fields_autoplaced yes)
-		(property "Reference" "C8"
+		(property "Reference" "C13"
 			(at 162.56 88.9 90)
 			(show_name no)
@@
 			(project "pwm_generator"
 				(path "/8c5142ba-d623-44cf-91e0-639551b20541/749c89d5-b92c-45c1-9dff-9c60a81aaaf0"
-					(reference "C8")
+					(reference "C13")
 					(unit 1)
 				)
@@
 		(in_pos_files yes)
 		(dnp no)
-		(property "Reference" "#PWR024"
+		(property "Reference" "#PWR029"
 			(at 146.05 74.93 0)
 			(hide yes)
@@
 			(project "pwm_generator"
 				(path "/8c5142ba-d623-44cf-91e0-639551b20541/749c89d5-b92c-45c1-9dff-9c60a81aaaf0"
-					(reference "#PWR024")
-					(unit 1)
-				)
+					(reference "#PWR029")
+					(unit 1)
+				)

Commit message: Uprava DPS generatoru - popisky
Connections:
- net ~{SAMPLING} renamed ~{TRIGGER}
Changed lines of the file:
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@@
 		)
 	)
-	(hierarchical_label "~{SAMPLING}"
+	(hierarchical_label "~{TRIGGER}"
 		(shape output)
 		(at 102.87 128.27 180)

Commit message: Pridany testpointy a jlcpcb bom reference
Parts:
- C10, C11, C12, C14: JLCPCB Part # (none) -> C49678
- C13: JLCPCB Part # (none) -> C7467177
- R11: JLCPCB Part # (none) -> C4382
- R12: JLCPCB Part # (none) -> C17772
- R13: JLCPCB Part # (none) -> C17414
- R14, R15: JLCPCB Part # (none) -> C17506
- U4: JLCPCB Part # (none) -> C193413
- U5: JLCPCB Part # (none) -> C96626
Changed lines of the file:
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@@
+			)
+		)
+		(property "JLCPCB Part #" "C49678"
+			(at 125.73 119.38 90)
+			(hide yes)
+			(show_name no)
+			(do_not_autoplace no)
+			(effects
+				(font
+					(size 1.27 1.27)
+				)
 			)
 		)
@@
 			)
 		)
+		(property "JLCPCB Part #" "C17414"
+			(at 132.08 107.95 90)
+			(hide yes)
+			(show_name no)
+			(do_not_autoplace no)
+			(effects
+				(font
+					(size 1.27 1.27)
+				)
+			)
+		)
 		(pin "1"
 		)
@@
 			)
 		)
+		(property "JLCPCB Part #" "C17506"
+			(at 162.56 107.95 90)
+			(hide yes)
+			(show_name no)
+			(do_not_autoplace no)
+			(effects
+				(font
+					(size 1.27 1.27)
+				)
+			)
+		)
 		(pin "1"
 		)
@@
 		)
 		(property "Description" "50-MHz, Zero-Crossover, Low-Distortion, High CMRR, RRI/O, Single-Supply, SOT-23-5"
+			(at 148.59 60.96 0)
+			(hide yes)
+			(show_name no)
+			(do_not_autoplace no)
+			(effects
+				(font
+					(size 1.27 1.27)
+				)
+			)
+		)
+		(property "JLCPCB Part #" "C96626"
 			(at 148.59 60.96 0)
 			(hide yes)
@@
 			)
 		)
+		(property "JLCPCB Part #" "C4382"
+			(at 132.08 80.01 90)
+			(hide yes)
+			(show_name no)
+			(do_not_autoplace no)
+			(effects
+				(font
+					(size 1.27 1.27)
+				)
+			)
+		)
 		(pin "1"
 		)
@@
 			)
 		)
+		(property "JLCPCB Part #" "C17772"
+			(at 132.08 96.52 90)
+			(hide yes)
+			(show_name no)
+			(do_not_autoplace no)
+			(effects
+				(font
+					(size 1.27 1.27)
+				)
+			)
+		)
 		(pin "1"
 		)
@@
 			)
 		)
+		(property "JLCPCB Part #" "C17506"
+			(at 162.56 125.73 90)
+			(hide yes)
+			(show_name no)
+			(do_not_autoplace no)
+			(effects
+				(font
+					(size 1.27 1.27)
+				)
+			)
+		)
 		(pin "1"
 		)
@@
 		)
 		(property "Description" "Unpolarized capacitor"
+			(at 162.56 134.62 0)
+			(hide yes)
+			(show_name no)
+			(do_not_autoplace no)
+			(effects
+				(font
+					(size 1.27 1.27)
+				)
+			)
+		)
+		(property "JLCPCB Part #" "C49678"
 			(at 162.56 134.62 0)
 			(hide yes)
@@
 			)
 		)
+		(property "JLCPCB Part #" "C193413"
+			(at 129.54 128.27 0)
+			(hide yes)
+			(show_name no)
+			(do_not_autoplace no)
+			(effects
+				(font
+					(size 1.27 1.27)
+				)
+			)
+		)
 		(pin "6"
 		)
@@
 		(property "Description" "Unpolarized capacitor"
 			(at 139.7 52.07 0)
+			(hide yes)
+			(show_name no)
+			(do_not_autoplace no)
+			(effects
+				(font
+					(size 1.27 1.27)
+				)
+			)
+		)
+		(property "JLCPCB Part #" "C49678"
+			(at 139.7 52.07 90)
 			(hide yes)
 			(show_name no)
@@
 			)
 		)
+		(property "JLCPCB Part #" "C49678"
+			(at 119.38 62.23 0)
+			(hide yes)
+			(show_name no)
+			(do_not_autoplace no)
+			(effects
+				(font
+					(size 1.27 1.27)
+				)
+			)
+		)
 		(pin "1"
 		)
@@
 			(hide yes)
 			(show_name no)
+			(do_not_autoplace no)
+			(effects
+				(font
+					(size 1.27 1.27)
+				)
+			)
+		)
+		(property "JLCPCB Part #" "C7467177"
+			(at 162.56 96.52 90)
+			(hide yes)
+			(show_name no)

Commit message: Doplnene testovaci body a popisky
Parts:
- renumbered R11 to R12, R12 to R13, R13 to R14, R14 to R15, R15 to R16
Changed lines of the file:
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@@
 		(dnp no)
 		(fields_autoplaced yes)
-		(property "Reference" "#PWR028"
+		(property "Reference" "#PWR030"
 			(at 146.05 54.61 0)
 			(hide yes)
@@
 			(project "pwm_generator"
 				(path "/8c5142ba-d623-44cf-91e0-639551b20541/749c89d5-b92c-45c1-9dff-9c60a81aaaf0"
-					(reference "#PWR028")
+					(reference "#PWR030")
 					(unit 1)
 				)
@@
 		(dnp no)
 		(fields_autoplaced yes)
-		(property "Reference" "#PWR027"
+		(property "Reference" "#PWR029"
 			(at 129.54 52.07 0)
 			(hide yes)
@@
 			(project "pwm_generator"
 				(path "/8c5142ba-d623-44cf-91e0-639551b20541/749c89d5-b92c-45c1-9dff-9c60a81aaaf0"
-					(reference "#PWR027")
+					(reference "#PWR029")
 					(unit 1)
 				)
@@
 		(dnp no)
 		(fields_autoplaced yes)
-		(property "Reference" "#PWR023"
+		(property "Reference" "#PWR025"
 			(at 115.57 119.38 0)
 			(hide yes)
@@
 			(project "pwm_generator"
 				(path "/8c5142ba-d623-44cf-91e0-639551b20541/749c89d5-b92c-45c1-9dff-9c60a81aaaf0"
-					(reference "#PWR023")
+					(reference "#PWR025")
 					(unit 1)
 				)
@@
 		(dnp no)
 		(fields_autoplaced yes)
-		(property "Reference" "R13"
+		(property "Reference" "R14"
 			(at 132.08 101.6 90)
 			(show_name no)
@@
 			(project "pwm_generator"
 				(path "/8c5142ba-d623-44cf-91e0-639551b20541/749c89d5-b92c-45c1-9dff-9c60a81aaaf0"
-					(reference "R13")
+					(reference "R14")
 					(unit 1)
 				)
@@
 		(dnp no)
 		(fields_autoplaced yes)
-		(property "Reference" "R14"
+		(property "Reference" "R15"
 			(at 162.56 101.6 90)
 			(show_name no)
@@
 			(project "pwm_generator"
 				(path "/8c5142ba-d623-44cf-91e0-639551b20541/749c89d5-b92c-45c1-9dff-9c60a81aaaf0"
-					(reference "R14")
+					(reference "R15")
 					(unit 1)
 				)
@@
 		(dnp no)
 		(fields_autoplaced yes)
-		(property "Reference" "R11"
+		(property "Reference" "R12"
 			(at 132.08 73.66 90)
 			(show_name no)
@@
 			(project "pwm_generator"
 				(path "/8c5142ba-d623-44cf-91e0-639551b20541/749c89d5-b92c-45c1-9dff-9c60a81aaaf0"
-					(reference "R11")
+					(reference "R12")
 					(unit 1)
 				)
@@
 		(dnp no)
 		(fields_autoplaced yes)
-		(property "Reference" "#PWR024"
+		(property "Reference" "#PWR026"
 			(at 129.54 144.78 0)
 			(hide yes)
@@
 			(project "pwm_generator"
 				(path "/8c5142ba-d623-44cf-91e0-639551b20541/749c89d5-b92c-45c1-9dff-9c60a81aaaf0"
-					(reference "#PWR024")
+					(reference "#PWR026")
 					(unit 1)
 				)
@@
 		(dnp no)
 		(fields_autoplaced yes)
-		(property "Reference" "R12"
+		(property "Reference" "R13"
 			(at 132.08 90.17 90)
 			(show_name no)
@@
 			(project "pwm_generator"
 				(path "/8c5142ba-d623-44cf-91e0-639551b20541/749c89d5-b92c-45c1-9dff-9c60a81aaaf0"
-					(reference "R12")
+					(reference "R13")
 					(unit 1)
 				)
@@
 		(dnp no)
 		(fields_autoplaced yes)
-		(property "Reference" "#PWR026"
+		(property "Reference" "#PWR028"
 			(at 132.08 144.78 0)
 			(hide yes)
@@
 			(project "pwm_generator"
 				(path "/8c5142ba-d623-44cf-91e0-639551b20541/749c89d5-b92c-45c1-9dff-9c60a81aaaf0"
-					(reference "#PWR026")
+					(reference "#PWR028")
 					(unit 1)
 				)
@@
 		(dnp no)
 		(fields_autoplaced yes)
-		(property "Reference" "#PWR022"
+		(property "Reference" "#PWR024"
 			(at 119.38 72.39 0)
 			(hide yes)
@@
 			(project "pwm_generator"
 				(path "/8c5142ba-d623-44cf-91e0-639551b20541/749c89d5-b92c-45c1-9dff-9c60a81aaaf0"
-					(reference "#PWR022")
+					(reference "#PWR024")
 					(unit 1)
 				)
@@
 		(dnp no)
 		(fields_autoplaced yes)
-		(property "Reference" "#PWR025"
+		(property "Reference" "#PWR027"
 			(at 132.08 121.92 0)
 			(hide yes)
@@
 			(project "pwm_generator"
 				(path "/8c5142ba-d623-44cf-91e0-639551b20541/749c89d5-b92c-45c1-9dff-9c60a81aaaf0"
-					(reference "#PWR025")
+					(reference "#PWR027")
 					(unit 1)
 				)
@@
 		(dnp no)
 		(fields_autoplaced yes)
-		(property "Reference" "R15"
+		(property "Reference" "R16"
 			(at 162.56 119.38 90)
 			(show_name no)
@@
 			(project "pwm_generator"
 				(path "/8c5142ba-d623-44cf-91e0-639551b20541/749c89d5-b92c-45c1-9dff-9c60a81aaaf0"
-					(reference "R15")
+					(reference "R16")
 					(unit 1)
 				)
@@
 		(dnp no)
 		(fields_autoplaced yes)
-		(property "Reference" "#PWR030"
+		(property "Reference" "#PWR032"
 			(at 162.56 144.78 0)
 			(hide yes)
@@
 			(project "pwm_generator"
 				(path "/8c5142ba-d623-44cf-91e0-639551b20541/749c89d5-b92c-45c1-9dff-9c60a81aaaf0"
-					(reference "#PWR030")
+					(reference "#PWR032")
 					(unit 1)
 				)
@@
 		(in_pos_files yes)
 		(dnp no)
-		(property "Reference" "#PWR029"
+		(property "Reference" "#PWR031"
 			(at 146.05 74.93 0)
 			(hide yes)
@@
 			(project "pwm_generator"
 				(path "/8c5142ba-d623-44cf-91e0-639551b20541/749c89d5-b92c-45c1-9dff-9c60a81aaaf0"
-					(reference "#PWR029")
-					(unit 1)
-				)
+					(reference "#PWR031")
+					(unit 1)
+				)
